Commit message: first commit

File: beetle_description/urdf/beetle.urdf (robot description, URDF)
Before this commit: robot beetle, 2 links, 3 joints
Links:
- added link laser_frame; collision cylinder length=0.04 radius=0.05; visual cylinder length=0.04 radius=0.05
Joints:
- added joint laser_joint: type fixed, parent base_link, child laser_frame, origin xyz=0 0 .25 rpy=0 0 0
